File: pcb_files/optical_encoder_pcb_test.kicad_sch (KiCad schematic)
At the start: 27 parts, among them J1 Conn_01x01_Pin, J10 Conn_DF13_malex06, J11 Conn_DF13_malex05, J12 Conn_DF13_malex05, J13 Conn_THT_padx04, J14 Conn_THT_padx04, J2 Conn_01x02_Pin, J3 Conn_01x04_Pin, J4 Conn_01x03_Pin, J5 Conn_01x04_Pin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

Commit message: Propositions de corrections v2.
Parts:
- removed J1: Conn_01x01_Pin, Connector_PinHeader_2.54mm:PinHeader_1x01_P2.54mm_Vertical, symbol Connector:Conn_01x01_Pin
- removed J11, J12: Conn_DF13_malex05, Connector_Hirose:Hirose_DF13-05P-1.25DS_1x05_P1.25mm_Horizontal, symbol Connector_Generic:Conn_01x05
- removed J2, J7, J8: Conn_01x02_Pin, Connector_PinHeader_2.54mm:PinHeader_1x02_P2.54mm_Vertical, symbol Connector:Conn_01x02_Pin
- removed J3: Conn_01x04_Pin, Connector_PinHeader_2.54mm:PinHeader_1x04_P2.54mm_Vertical, symbol Connector:Conn_01x04_Pin
- removed J6: Conn_01x03_Pin, Connector_PinHeader_2.54mm:PinHeader_1x03_P2.54mm_Vertical, symbol Connector:Conn_01x03_Pin
- added C7: 1uF, Capacitor_SMD:C_0402_1005Metric, symbol Device:C
- added C8: 100nF, Capacitor_SMD:C_0402_1005Metric, symbol Device:C
- added C9: 10uF, Capacitor_SMD:C_0402_1005Metric, symbol Device:C
- added J2: Conn_01x05_Pin, Connector_PinHeader_2.54mm:PinHeader_1x05_P2.54mm_Vertical, symbol Connector:Conn_01x05_Pin
- added J4: Conn_01x04_Pin, Connector_PinHeader_2.54mm:PinHeader_1x04_P2.54mm_Vertical, symbol Connector:Conn_01x04_Pin
- added R6, R7: 10K, Resistor_SMD:R_0805_2012Metric_Pad1.20x1.40mm_HandSolder, symbol Device:R
- added U2: AMS1117-3.3, Package_TO_SOT_SMD:SOT-223-3_TabPin2, symbol Regulator_Linear:AMS1117-3.3
- renumbered J4 to J1
Connections:
- net CFG0 is gone; now on net GND: Ic-pz2656.1 (CFG(0))
- net CFG1 is gone; now on net GND: Ic-pz2656.32 (CFG(1))
- net CFG2 is gone; now on net GND: Ic-pz2656.31 (CFG(2))
- net VDDA is gone; now on net +5V: C3.2, C4.2, Ic-pz2656.30 (VDDA)
- net GND: now also J1.2 (Pin_2), J5.4 (Pin_4), C7.2, C8.2, C9.2, J2.1 (Pin_1), J4.4 (Pin_4), R6.2, U2.1 (GND)
- net ACL: no longer names the net of Ic-pz2656.18 (ACL)
- net ADA: no longer names the net of Ic-pz2656.19 (ADA)
- net ERR_IN: no longer names the net of Ic-pz2656.20 (GPIO(1))
- net PA0 renamed SPI_MISO
- net SPI_MISO: now also J2.5 (Pin_5), R6.1
- net PA1 renamed SPI_MOSI
- net SPI_MOSI: now also J2.4 (Pin_4)
- net PA2 renamed SPI_SCLK
- net SPI_SCLK: now also J2.3 (Pin_3)
- net PA3 renamed SPI_~{CS}
- net SPI_~{CS}: now also J2.2 (Pin_2), R7.1
- net PB0 renamed +5V
- net +5V: now also J10.2 (Pin_2), C7.1, C8.1, U2.3 (VI); no longer Ic-pz2656.17 (PORTB(0))
- net PB1 renamed BiSS_SLI
- net BiSS_SLI: now also J4.2 (Pin_2); no longer J1.2 (Pin_2)
- net PB2 renamed +3.3V
- net +3.3V: now also C1.2, C2.2, C6.2, Ic-pz2656.14 (VDDIO), J9.2 (Pin_2), R1.2, R2.2, R3.1, U1.4 (VCC), C9.1, R7.2, U2.2 (VO); no longer Ic-pz2656.15 (PORTB(2))
- net PC0 renamed Z
- net PC1 renamed B
- net PC2 renamed A
- removed net PC3: Ic-pz2656.23 (PORTC(3)), J10.6 (Pin_6), J5.4 (Pin_4)
- net RDY: no longer names the net of Ic-pz2656.21 (GPIO(0))
- removed net VDDIO: C1.2, C2.2, C6.2, Ic-pz2656.14 (VDDIO), J10.2 (Pin_2), J9.2 (Pin_2), R1.2, R2.2, R3.1, U1.4 (VCC)
- new net BiSS_MA: Ic-pz2656.15 (PORTB(2)), J4.3 (Pin_3)
- new net BiSS_SLO: Ic-pz2656.17 (PORTB(0)), J4.1 (Pin_1)
- no-connect marks 0 -> 5
Other:
- note added: "CFG0/CFG1/CFG2 -> to GNDIO PortA = SPI PortB = BiSS/SSI PortC = ABZ ---------------------- PortA.3 = /CS PortA.2 = SCLK PortA.1 = MOSI PortA.0 = MISO (mettre resistance 10k en MOSI et GNDIO) ---------------------- PortB.2 = MA PortB.1 = SLI PortB.0 = SLO ---------------------- PortC.2 = A PortC.1 = B PortC.0 = Z"
- note added: "Pour gagner en place Remplacer C1, C2, C3, C4 & C5 par C7 & C8 (0402 au lieu de 0805)"
- note added: "Pour gagner en place on peut aussi remplacer les résistances en 0402 au lieu de 0805"
- note added: "Qu'est ce que c'est?"
- note added: "Remplacer J10, 6 pins par un 5 pins. Supprimer PC3. Remplacer VDDIO (+3.3V) par VDDA (+5.0V)"
- note added: "U2 est un regulateur. Il va passer la tension de 5.0V à 3.3V"
- moved on the sheet: C6, J1, J13, J14, J5

Commit message: Story 2 : add voltage regulator, fix configuration, modify connectors
Parts:
- removed J10: Conn_DF13_malex06, Connector_Hirose:Hirose_DF13-06P-1.25DS_1x06_P1.25mm_Horizontal, symbol Connector_Generic:Conn_01x06
- removed J13, J14: Conn_THT_padx04, Connector_PinHeader_2.54mm:PinHeader_1x04_P2.54mm_Vertical, symbol Connector:Conn_01x04_Socket
- added J6: Conn_DF13_male_01x05, Connector_Hirose:Hirose_DF13-05P-1.25DSA_1x05_P1.25mm_Vertical, symbol Connector_Generic:Conn_01x05
- added J7: Conn_AMASS_male_01x03, Connector_AMASS:AMASS_MR30PW-M_1x03_P3.50mm_Horizontal, symbol Connector_Generic:Conn_01x03
- added J8: Conn_01x03_Pin, Connector_PinHeader_2.54mm:PinHeader_1x03_P2.54mm_Vertical, symbol Connector:Conn_01x03_Pin
- C1, C2, C3, C4, C5, C6: footprint Capacitor_SMD:C_0805_2012Metric_Pad1.18x1.45mm_HandSolder -> Capacitor_SMD:C_0402_1005Metric_Pad0.74x0.62mm_HandSolder
- C7, C8, C9: footprint Capacitor_SMD:C_0402_1005Metric -> Capacitor_SMD:C_0402_1005Metric_Pad0.74x0.62mm_HandSolder
- J5: renamed from J9; value Conn_DF13_malex06 -> Conn_DF13_male_01x06
- R1, R2, R3, R4, R5, R6, R7: footprint Resistor_SMD:R_0805_2012Metric_Pad1.20x1.40mm_HandSolder -> Resistor_SMD:R_0402_1005Metric_Pad0.72x0.64mm_HandSolder
- renumbered J4 to J3, J5 to J4
Connections:
- net +5V: now also J6.2 (Pin_2)
- net A: now also J6.5 (Pin_5)
- net B: now also J6.4 (Pin_4)
- net GND: now also J6.1 (Pin_1)
- net Z: now also J6.3 (Pin_3)
- new net P1: J7.1 (Pin_1), J8.1 (Pin_1)
- new net P2: J7.2 (Pin_2), J8.2 (Pin_2)
- new net P3: J7.3 (Pin_3), J8.3 (Pin_3)
Other:
- note added: "Remplacer J6, 6 pins par un 5 pins. Supprimer PC3. Remplacer VDDIO (+3.3V) par VDDA (+5.0V)"
- note added: "utiliser des AMASS en entrée et un pad traversant pour soudure en sortie. connexions : P1,P2,P3 du moteur"
- note removed: "Qu'est ce que c'est?"
- note removed: "Remplacer J10, 6 pins par un 5 pins. Supprimer PC3. Remplacer VDDIO (+3.3V) par VDDA (+5.0V)"
- moved on the sheet: J5
