File: pcb_files/optical_encoder-pcb_test/optical_encoder_pcb_test.kicad_pcb (KiCad board)
At the start: 2 copper layers, 53.7 x 54.9 mm, 33 parts, among them J1 Conn_01x03_Pin, J2 Conn_01x05_Pin, J3 Conn_01x04_Pin, J4 Conn_01x04_Pin, J5 Conn_DF13_male_01x06, J6 Conn_DF13_male_01x05, J7 Conn_AMASS_male_01x03, J8 Conn_01x03_Pin, U1 AT24CS16-STUM, U2 AMS1117-3.3

Commit message: Double phase traces, C7-C8-C9 switched to front face, C5-R3 moved
Parts:
- C5, C7, C8, C9, R3: moved to F.Cu
- moved C6 10.0 mm to (117.2, 105.3), turned to 90 degrees
- moved C7 9.17 mm to (106.5, 103.4), turned to -90 degrees
- moved R3 8.02 mm to (126.8, 108.1)
- moved C8 7.90 mm to (108.3, 103.4), turned to -90 degrees
- moved C9 7.48 mm to (106.5, 107.1), turned to -90 degrees
- moved J3 5.20 mm to (131.2, 111.5), turned to 180 degrees
- moved REF** 2.77 mm to (136.4, 128.4)
- moved R6 2.40 mm to (115.2, 118.4)
- moved C5 0.91 mm to (118.5, 117.4)
- moved J1 0.10 mm to (114.0, 108.0)
Routing:
- net +3.3V: track 61.9 -> 68.6 mm, vias 3 -> 2
- net +5V: track 26.9 -> 31.8 mm, vias 2 -> 1
- net /BiSS_SLO: track 4.67 -> 9.47 mm
- net Net-(Ic-pz2656-NRES): track 5.01 -> 9.64 mm
- net /BiSS_SLI: track 7.83 -> 9.41 mm
- net /BiSS_MA: track 11.7 -> 10.3 mm
- net /SPI_MISO: track 17.5 -> 18.9 mm
- net Net-(Ic-pz2656-C1V8): track 2.55 -> 2.90 mm, vias 1 -> 0
- added copper zone on F.Cu, net /P1
- added copper zone on F.Cu, net /P2
- added copper zone on F.Cu, net /P3
